Commit message: Initial commit with Kinect and robot setup

File: install/rmis_description/share/rmis_description/urdf/rmis_robot.urdf (robot description, URDF)
Before this commit: robot rmis_robot, 23 links, 22 joints
Links:
- link head_link_k: geometry visual mesh filename=package://rmis_description/meshes/dae/27-1a.001.dae scale=1.00000 1.00000 1.00000
- link l_ankle_link_k: geometry visual mesh filename=package://rmis_description/meshes/dae/Cube.001.dae scale=0.77000 0.81000 1.00000; visual mesh filename=package://rmis_description/meshes/dae/u_bracket.003.dae scale=1.00000 1.00000 1.00000
- link l_arm_link_k1: geometry visual mesh filename=package://rmis_description/meshes/dae/u_bracket.015.dae scale=1.00000 1.00000 1.00000
- link l_arm_link_k2: geometry visual mesh filename=package://rmis_description/meshes/dae/Cube.019.dae scale=2.00000 18.36721 18.36721
- link l_hand_link_k: geometry visual mesh filename=package://rmis_description/meshes/dae/offset_bracket.001.dae scale=1.00000 1.00000 1.00000
- link l_hip_link_k: geometry visual mesh filename=package://rmis_description/meshes/dae/Hub_torque.dae scale=1.00000 1.00000 1.00000; visual mesh filename=package://rmis_description/meshes/dae/u_bracket.004.dae scale=1.00000 1.00000 1.00000
- link l_leg_base_link_k: geometry visual mesh filename=package://rmis_description/meshes/dae/Hub_torque.008.dae scale=1.00000 1.00000 1.00000
- link l_lower_leg_link_k: geometry visual mesh filename=package://rmis_description/meshes/dae/Cube.017.dae scale=2.00000 9.66935 9.66936; visual mesh filename=package://rmis_description/meshes/dae/u_bracket.001.dae scale=1.00000 1.00000 1.00000
- link l_shoulder_base_link_k: geometry visual mesh filename=package://rmis_description/meshes/dae/u_bracket.011.dae scale=1.00000 1.00000 1.00000
- link l_shoulder_child_link_k: geometry visual mesh filename=package://rmis_description/meshes/dae/Hub_torque.020.dae scale=1.00000 1.00000 1.00000
- link l_upper_leg_link_k: geometry visual mesh filename=package://rmis_description/meshes/dae/Cube.005.dae scale=2.00000 9.66936 9.66936; visual mesh filename=package://rmis_description/meshes/dae/Hub_torque.036.dae scale=1.00000 1.00000 1.00000
- link neck_link_k: geometry visual mesh filename=package://rmis_description/meshes/dae/Hub_torque.002.dae scale=1.00000 1.00000 1.00000
- link r_ankle_link_k: geometry visual mesh filename=package://rmis_description/meshes/dae/Cube.029.dae scale=0.77000 0.81000 1.00000; visual mesh filename=package://rmis_description/meshes/dae/u_bracket.012.dae scale=1.00000 1.00000 1.00000
- link r_arm_link_k1: geometry visual mesh filename=package://rmis_description/meshes/dae/u_bracket.014.dae scale=1.00000 1.00000 1.00000
- link r_arm_link_k2: geometry visual mesh filename=package://rmis_description/meshes/dae/Cube.021.dae scale=2.00000 18.36721 18.36721
- link r_hand_link_k: geometry visual mesh filename=package://rmis_description/meshes/dae/offset_bracket.003.dae scale=1.00000 1.00000 1.00000
- link r_hip_link_k: geometry visual mesh filename=package://rmis_description/meshes/dae/Hub_torque.011.dae scale=1.00000 1.00000 1.00000; visual mesh filename=package://rmis_description/meshes/dae/u_bracket.005.dae scale=1.00000 1.00000 1.00000
- link r_leg_base_link_k: geometry visual mesh filename=package://rmis_description/meshes/dae/Hub_torque.010.dae scale=1.00000 1.00000 1.00000
- link r_lower_leg_link_k: geometry visual mesh filename=package://rmis_description/meshes/dae/Cube.023.dae scale=2.00000 9.66936 9.66936; visual mesh filename=package://rmis_description/meshes/dae/u_bracket.007.dae scale=1.00000 1.00000 1.00000
- link r_shoulder_base_link_k: geometry visual mesh filename=package://rmis_description/meshes/dae/u_bracket.010.dae scale=1.00000 1.00000 1.00000
- link r_shoulder_child_link_k: geometry visual mesh filename=package://rmis_description/meshes/dae/Cube.007.dae scale=2.00000 9.66936 9.66936
- link r_upper_leg_link_k: geometry visual mesh filename=package://rmis_description/meshes/dae/Cube.008.dae scale=2.00000 9.66936 9.66936; visual mesh filename=package://rmis_description/meshes/dae/Hub_torque.035.dae scale=1.00000 1.00000 1.00000
- link root_link_k: geometry visual mesh filename=package://rmis_description/meshes/dae/Cube.020.dae scale=1.01000 1.00000 1.00000
Joints:
- joint r_ankle_link_k_joint: origin xyz=67.37613 -0.01323 -0.03973 rpy=-0.00000 -0.00000 0.00000 -> xyz=67.37610 -0.01323 -0.03973 rpy=-0.00000 0.00000 -0.00000
- joint r_lower_leg_link_k_joint: origin xyz=66.92873 -0.84708 -0.12632 rpy=-0.00000 0.00000 -0.01530 -> xyz=66.82124 3.88529 -0.12632 rpy=0.00000 0.00000 0.05543

Commit message: rmis_gazebo_environment

File: install/rmis_description/share/rmis_description/urdf/rmis_robot.urdf (robot description, URDF)
Before this commit: robot rmis_robot, 23 links, 22 joints
Links:
- link head_link_k: mass None -> 0.001; geometry collision box size=0.05 0.05 0.05; visual mesh filename=package://rmis_description/meshes/dae/27-1a.001.dae scale=0.001 0.001 0.001
- link l_ankle_link_k: mass None -> 0.001; geometry collision box size=0.05 0.05 0.05; collision box size=0.05 0.05 0.05
- link l_arm_link_k1: mass None -> 0.001; geometry collision box size=0.05 0.05 0.05; visual mesh filename=package://rmis_description/meshes/dae/u_bracket.015.dae scale=0.001 0.001 0.001
- link l_arm_link_k2: mass None -> 0.001; geometry collision box size=0.05 0.05 0.05; visual mesh filename=package://rmis_description/meshes/dae/Cube.019.dae scale=0.002 0.01836721 0.01836721
- link l_hand_link_k: mass None -> 0.001; geometry collision box size=0.05 0.05 0.05; visual mesh filename=package://rmis_description/meshes/dae/offset_bracket.001.dae scale=0.001 0.001 0.001
- link l_hip_link_k: mass None -> 0.001; geometry collision box size=0.05 0.05 0.05; collision box size=0.05 0.05 0.05
- link l_leg_base_link_k: mass None -> 0.002; geometry collision box size=0.05 0.05 0.05; visual mesh filename=package://rmis_description/meshes/dae/Hub_torque.008.dae scale=0.001 0.001 0.001
- link l_lower_leg_link_k: mass None -> 0.001; geometry collision box size=0.05 0.05 0.05; collision box size=0.05 0.05 0.05
- link l_shoulder_base_link_k: mass None -> 0.001; geometry collision box size=0.05 0.05 0.05; visual mesh filename=package://rmis_description/meshes/dae/u_bracket.011.dae scale=0.001 0.001 0.001
- link l_shoulder_child_link_k: mass None -> 0.001; geometry collision box size=0.05 0.05 0.05; visual mesh filename=package://rmis_description/meshes/dae/Hub_torque.020.dae scale=0.001 0.001 0.001
- link l_upper_leg_link_k: mass None -> 0.001; geometry collision box size=0.05 0.05 0.05; collision box size=0.05 0.05 0.05
- link neck_link_k: mass None -> 0.001; geometry collision box size=0.05 0.05 0.05; visual mesh filename=package://rmis_description/meshes/dae/Hub_torque.002.dae scale=0.001 0.001 0.001
- link r_ankle_link_k: mass None -> 0.001; geometry collision box size=0.05 0.05 0.05; collision box size=0.05 0.05 0.05
- link r_arm_link_k1: mass None -> 0.001; geometry collision box size=0.05 0.05 0.05; visual mesh filename=package://rmis_description/meshes/dae/u_bracket.014.dae scale=0.001 0.001 0.001
- link r_arm_link_k2: mass None -> 0.001; geometry collision box size=0.05 0.05 0.05; visual mesh filename=package://rmis_description/meshes/dae/Cube.021.dae scale=0.002 0.01836721 0.01836721
- link r_hand_link_k: mass None -> 0.001; geometry collision box size=0.05 0.05 0.05; visual mesh filename=package://rmis_description/meshes/dae/offset_bracket.003.dae scale=0.001 0.001 0.001
- link r_hip_link_k: mass None -> 0.001; geometry collision box size=0.05 0.05 0.05; collision box size=0.05 0.05 0.05
- link r_leg_base_link_k: mass None -> 0.002; geometry collision box size=0.05 0.05 0.05; visual mesh filename=package://rmis_description/meshes/dae/Hub_torque.010.dae scale=0.001 0.001 0.001
- link r_lower_leg_link_k: mass None -> 0.001; geometry collision box size=0.05 0.05 0.05; collision box size=0.05 0.05 0.05
- link r_shoulder_base_link_k: mass None -> 0.001; geometry collision box size=0.05 0.05 0.05; visual mesh filename=package://rmis_description/meshes/dae/u_bracket.010.dae scale=0.001 0.001 0.001
- link r_shoulder_child_link_k: mass None -> 0.001; geometry collision box size=0.05 0.05 0.05; visual mesh filename=package://rmis_description/meshes/dae/Cube.007.dae scale=0.002 0.00966936 0.00966936
- link r_upper_leg_link_k: mass None -> 0.001; geometry collision box size=0.05 0.05 0.05; collision box size=0.05 0.05 0.05
- link root_link_k: mass None -> 0.005; geometry collision box size=0.05 0.05 0.05; visual mesh filename=package://rmis_description/meshes/dae/Cube.020.dae scale=0.001 0.001 0.001
Joints:
- joint head_link_k_joint: origin xyz=-19.46497 -2.05624 35.79721 rpy=0.00000 -1.57080 0.00000 -> xyz=-0.01946497 -0.00205624 0.03579721 rpy=0.00000 -1.57080 0.00000
- joint l_ankle_link_k_joint: origin xyz=-66.90888 -0.02077 -0.09073 rpy=-0.00000 -0.00000 0.00000 -> xyz=-0.06690888 -0.00002077 -0.00009073 rpy=-0.00000 -0.00000 0.00000
- joint l_arm_link_k1_joint: origin xyz=0.52979 82.22321 -18.24224 rpy=1.57080 -0.00000 3.14159 -> xyz=0.00052979 0.08222321 -0.01824224 rpy=1.57080 -0.00000 3.14159
- joint l_arm_link_k2_joint: origin xyz=20.58876 0.13071 35.95849 rpy=-0.00000 1.57080 0.00000 -> xyz=0.02058876 0.00013071 0.03595849 rpy=-0.00000 1.57080 0.00000
- joint l_hand_link_k_joint: origin xyz=-68.90010 27.15716 -22.74708 rpy=-1.57080 1.57080 0.00000 -> xyz=-0.06890010 0.02715716 -0.02274708 rpy=-1.57080 1.57080 0.00000
- joint l_hip_link_k_joint: origin xyz=-9.85686 32.56039 24.17409 rpy=1.57080 -0.00000 -3.14159 -> xyz=-0.00985686 0.03256039 0.02417409 rpy=1.57080 -0.00000 -3.14159
- joint l_leg_base_link_k_joint: origin xyz=-48.34199 -18.27487 -131.41250 rpy=-3.14159 0.00000 -3.09779 -> xyz=-0.04834199 -0.01827487 -0.13141250 rpy=-3.14159 0.00000 -3.09779
- joint l_lower_leg_link_k_joint: origin xyz=-66.85407 0.06718 -1.14178 rpy=0.00000 0.00000 -0.00000 -> xyz=-0.06685407 0.00006718 -0.00114178 rpy=0.00000 0.00000 -0.00000
- joint l_shoulder_base_link_k_joint: origin xyz=-97.63426 -11.24756 51.72586 rpy=0.00000 -1.57080 0.00000 -> xyz=-0.09763426 -0.01124756 0.05172586 rpy=0.00000 -1.57080 0.00000
- joint l_shoulder_child_link_k_joint: origin xyz=0.91104 22.00416 35.45252 rpy=-1.57080 1.57080 0.00000 -> xyz=0.00091104 0.02200416 0.03545252 rpy=-1.57080 1.57080 0.00000
- joint l_upper_leg_link_k_joint: origin xyz=-32.91063 45.17123 -29.68048 rpy=1.57080 0.00000 -1.57080 -> xyz=-0.03291063 0.04517123 -0.02968048 rpy=1.57080 0.00000 -1.57080
- joint neck_link_k_joint: origin xyz=0.00000 -0.00000 83.06138 rpy=0.00000 0.00000 0.00000 -> xyz=0.00000 -0.00000 0.08306138 rpy=0.00000 0.00000 0.00000
- joint r_ankle_link_k_joint: origin xyz=67.37610 -0.01323 -0.03973 rpy=-0.00000 0.00000 -0.00000 -> xyz=0.06737610 -0.00001323 -0.00003973 rpy=-0.00000 0.00000 -0.00000
- joint r_arm_link_k1_joint: origin xyz=-0.22886 82.21970 -16.19683 rpy=-1.57080 0.00000 -0.00000 -> xyz=-0.00022886 0.08221970 -0.01619683 rpy=-1.57080 0.00000 -0.00000
- joint r_arm_link_k2_joint: origin xyz=18.95558 0.17086 35.89349 rpy=-2.28313 -1.57080 -0.85846 -> xyz=0.01895558 0.00017086 0.03589349 rpy=-2.28313 -1.57080 -0.85846
- joint r_hand_link_k_joint: origin xyz=68.59900 25.65830 -21.54085 rpy=-1.57080 -1.57080 0.00000 -> xyz=0.06859900 0.02565830 -0.02154085 rpy=-1.57080 -1.57080 0.00000
- joint r_hip_link_k_joint: origin xyz=-9.72866 -33.20288 24.18766 rpy=1.57080 0.00000 0.00000 -> xyz=-0.00972866 -0.03320288 0.02418766 rpy=1.57080 0.00000 0.00000
- joint r_leg_base_link_k_joint: origin xyz=48.64802 -18.52139 -131.39921 rpy=3.14159 0.00000 0.00000 -> xyz=0.04864802 -0.01852139 -0.13139921 rpy=3.14159 0.00000 0.00000
- joint r_lower_leg_link_k_joint: origin xyz=66.82124 3.88529 -0.12632 rpy=0.00000 0.00000 0.05543 -> xyz=0.06682124 0.00388529 -0.00012632 rpy=0.00000 0.00000 0.05543
- joint r_shoulder_base_link_k_joint: origin xyz=94.01596 -11.07213 51.94397 rpy=-0.00000 1.57080 0.00000 -> xyz=0.09401596 -0.01107213 0.05194397 rpy=-0.00000 1.57080 0.00000
- joint r_shoulder_child_link_k_joint: origin xyz=-0.69766 20.14315 39.18026 rpy=-1.57080 -1.57080 0.00000 -> xyz=-0.00069766 0.02014315 0.03918026 rpy=-1.57080 -1.57080 0.00000
- joint r_upper_leg_link_k_joint: origin xyz=31.79766 45.01670 -30.11760 rpy=1.57080 0.00000 1.57080 -> xyz=0.03179766 0.04501670 -0.03011760 rpy=1.57080 0.00000 1.57080
